File: hardware/sd_board.kicad_pcb (KiCad board)
At the start: 2 copper layers, 50.8 x 38.1 mm, 13 parts, among them J1 Screw_Terminal_01x03, SW1 SW_SPST, SW2 SW_SPST, U1 PIC16F18346-SS_0, U2 VL53L1CXV0FY1

Commit message: much better layout, need leds still though
Parts:
- moved J1 32.6 mm to (140.5, 67.3), turned to 180 degrees
- moved C2 15.1 mm to (145.5, 71.4)
- moved SW1 11.5 mm to (130.8, 87.9), turned to 180 degrees
- moved C4 11.3 mm to (150.4, 71.6), turned to 0 degrees
- moved SW2 10.4 mm to (144.3, 87.9)
- moved U2 9.04 mm to (150.4, 75.4), turned to 270 degrees
- moved R1 1.61 mm to (145.5, 76.7), turned to 180 degrees
- moved C3 1.52 mm to (136.7, 81.3)
- moved C5 1.52 mm to (136.7, 82.8)
- moved U1 1.52 mm to (136.7, 76.2)
- moved R2 0.57 mm to (145.5, 73.9), turned to 180 degrees
Routing:
- net VCC: track 50.5 -> 0.00 mm, vias 2 -> 0
- net Net-(J1-Pad3): track 45.2 -> 0.00 mm
- net Net-(J1-Pad2): track 35.9 -> 0.00 mm
- net XSHUT: track 34.9 -> 0.00 mm, vias 2 -> 0
- net INT: track 29.0 -> 0.00 mm
- net Net-(J2-Pad1): track 26.4 -> 0.00 mm, vias 2 -> 0
- net Net-(J2-Pad5): track 22.1 -> 0.00 mm, vias 2 -> 0
- net Net-(J2-Pad4): track 18.9 -> 0.00 mm, vias 2 -> 0
- net SDA: track 4.94 -> 0.00 mm
- net SCL: track 4.58 -> 0.00 mm
Other:
- board size 50.8 x 38.1 mm -> 39.4 x 27.9 mm
